File: hardware/ch570funprog.kicad_pcb (KiCad board)
At the start: 2 copper layers, 34.5 x 12.4 mm, 22 parts, among them J1 USB_C_Receptacle_USB2.0, J2 PGM, J3 DEVPGM, Q1 PMOS-SI2301CDS-T1-GE3, U1 USBLC6-2SC6, U2 AMS1117-3.3, U3 CH570Q, Y1 32M

Commit message: Bump.
Routing:
- net GND: vias 34 -> 35
Changed lines of the file:
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@@
 	)
 	(segment
+		(start 143.360242 82.6)
+		(end 143.35 82.88)
+		(width 0.2)
+		(layer "F.Cu")
+		(net 1)
+	)
+	(segment
 		(start 130.08 78.79)
 		(end 129 78.79)
@@
 	(segment
 		(start 143.388409 81.83)
-		(end 143.35 82.88)
+		(end 143.360242 82.6)
 		(width 0.2)
 		(layer "F.Cu")
@@
 	)
 	(via
+		(at 143.360242 82.6)
+		(size 0.6)
+		(drill 0.3)
+		(layers "F.Cu" "B.Cu")
+		(net 1)
+	)
+	(via
 		(at 150.91 81.88)
 		(size 0.6)
@@
 	)
 	(via
-		(at 145.39 81.71)
+		(at 144.92 80.96)
 		(size 0.6)
 		(drill 0.3)
@@
 		(start 150.71 80.6)
 		(end 150.76 80.11)
-		(width 0.2)
+		(width 0.25)
 		(layer "F.Cu")
 		(net 4)
@@
 		(start 140.835 82.53)
 		(end 141.89 82.48)
-		(width 0.2)
+		(width 0.25)
 		(layer "F.Cu")
 		(net 4)
@@
 	)
 	(segment
-		(start 149.96 79.96)
+		(start 153.29 82.29)
 		(end 150.71 80.6)
-		(width 0.2)
+		(width 0.25)
 		(layer "B.Cu")
 		(net 4)
 	)
 	(segment
-		(start 153.29 82.29)
-		(end 150.71 80.6)
-		(width 0.2)
+		(start 141.89 82.48)
+		(end 142.46 81.84)
+		(width 0.25)
 		(layer "B.Cu")
 		(net 4)
 	)
 	(segment
-		(start 142.36233 82.772751)
-		(end 145.57 82.83)
-		(width 0.2)
+		(start 149.78 79.56)
+		(end 150.71 80.6)
+		(width 0.25)
 		(layer "B.Cu")
 		(net 4)
 	)
 	(segment
-		(start 145.57 82.83)
-		(end 147.5 80.38)
-		(width 0.2)
+		(start 142.46 81.84)
+		(end 145.26 81.57)
+		(width 0.25)
 		(layer "B.Cu")
 		(net 4)
 	)
 	(segment
-		(start 147.5 80.38)
-		(end 148.34 79.9)
-		(width 0.2)
+		(start 145.26 81.57)
+		(end 147.31 79.87)
+		(width 0.25)
 		(layer "B.Cu")
 		(net 4)
 	)
 	(segment
-		(start 141.89 82.48)
-		(end 142.36233 82.772751)
-		(width 0.2)
+		(start 147.31 79.87)
+		(end 148.12 79.52)
+		(width 0.25)
 		(layer "B.Cu")
 		(net 4)
 	)
 	(segment
-		(start 148.34 79.9)
-		(end 149.96 79.96)
-		(width 0.2)
+		(start 148.12 79.52)
+		(end 149.78 79.56)
+		(width 0.25)
 		(layer "B.Cu")
 		(net 4)
@@
 		(start 140.835 83.03)
 		(end 141.25 83.04)
-		(width 0.2)
+		(width 0.25)
 		(layer "F.Cu")
 		(net 6)
 	)
 	(segment
-		(start 148.99 81.17)
-		(end 150.89 81.21)
-		(width 0.2)
+		(start 150.91 81.23)
+		(end 153.29 79.75)
+		(width 0.25)
 		(layer "F.Cu")
 		(net 6)
 	)
 	(segment
-		(start 147.4 81.51)
-		(end 148.99 81.17)
-		(width 0.2)
+		(start 147.448252 81.288252)
+		(end 148.42 81.3)
+		(width 0.25)
 		(layer "F.Cu")
 		(net 6)
@@
 		(start 141.25 83.04)
 		(end 141.41 83.14)
-		(width 0.2)
+		(width 0.25)
 		(layer "F.Cu")
 		(net 6)
 	)
 	(segment
-		(start 150.89 81.21)
-		(end 153.29 79.75)
-		(width 0.2)
+		(start 148.42 81.3)
+		(end 150.91 81.23)
+		(width 0.25)
 		(layer "F.Cu")
 		(net 6)
@@
 	(segment
 		(start 146.65 80.05)
-		(end 147.4 81.51)
-		(width 0.2)
+		(end 147.448252 81.288252)
+		(width 0.22)
 		(layer "F.Cu")
 		(net 6)
@@
 	)
 	(via
-		(at 147.4 81.51)
+		(at 147.448252 81.288252)
 		(size 0.6)
 		(drill 0.3)
@@
 	)
 	(segment
-		(start 145.74 83.29)
+		(start 142.14 83.34)
 		(end 141.41 83.14)
-		(width 0.2)
+		(width 0.25)
 		(layer "B.Cu")
 		(net 6)
 	)
 	(segment
-		(start 147.4 81.51)
-		(end 145.74 83.29)
-		(width 0.2)
+		(start 147 81.65)
+		(end 145.76 82.8)
+		(width 0.25)
+		(layer "B.Cu")
+		(net 6)
+	)
+	(segment
+		(start 145.76 82.8)
+		(end 143.3 83.26)
+		(width 0.25)
+		(layer "B.Cu")
+		(net 6)
+	)
+	(segment
+		(start 143.3 83.26)
+		(end 142.14 83.34)
+		(width 0.25)
+		(layer "B.Cu")
+		(net 6)
+	)
+	(segment
+		(start 147.448252 81.288252)
+		(end 147 81.65)
+		(width 0.25)
 		(layer "B.Cu")
 		(net 6)
@@
 	)
 	(zone
+		(net 6)
+		(net_name "SWD")
+		(layer "F.Cu")
+		(name "$teardrop_padvia$")
+		(hatch none 0.1)
+		(priority 30027)
+		(attr
+			(teardrop
+				(type padvia)
+			)
+		)
+		(connect_pads yes
+			(clearance 0)
+		)
+		(min_thickness 0.0254)
+		(filled_areas_thickness no)
+		(fill yes
+			(thermal_gap 0.5)
+			(thermal_bridge_width 0.5)
+			(island_removal_mode 1)
+			(island_area_min 10)
+		)
+		(polygon
+			(pts
+				(xy 146.899591 80.640183) (xy 147.084498 80.52098) (xy 146.92 79.970512) (xy 146.649459 80.04916)
+				(xy 146.53505 80.37)
+			)
+		)
+	)
+	(zone
 		(net 3)
 		(net_name "+5V")
@@
 		(name "$teardrop_padvia$")
 		(hatch none 0.1)
-		(priority 30056)
+		(priority 30055)
 		(attr
 			(teardrop
@@
 		(name "$teardrop_padvia$")
 		(hatch none 0.1)
-		(priority 30055)
+		(priority 30054)
 		(attr
 			(teardrop
@@
 	)
 	(zone
-		(net 6)
-		(net_name "SWD")
-		(layer "F.Cu")
-		(name "$teardrop_padvia$")
-		(hatch none 0.1)
-		(priority 30027)
-		(attr
-			(teardrop
-				(type padvia)
-			)
-		)
-		(connect_pads yes
-			(clearance 0)
-		)
-		(min_thickness 0.0254)
-		(filled_areas_thickness no)
-		(fill yes
-			(thermal_gap 0.5)
-			(thermal_bridge_width 0.5)
-			(island_removal_mode 1)
-			(island_area_min 10)
-		)
-		(polygon
-			(pts
-				(xy 146.846082 80.650555) (xy 147.023982 80.559168) (xy 146.92 79.984705) (xy 146.649544 80.049111)
-				(xy 146.510369 80.369079)
-			)
-		)
-	)
-	(zone
 		(net 14)
 		(net_name "PSWITCHED")
@@
 	)
 	(zone
-		(net 6)
-		(net_name "SWD")
-		(layer "F.Cu")
-		(name "$teardrop_padvia$")
-		(hatch none 0.1)
-		(priority 30057)
-		(attr
-			(teardrop
-				(type padvia)
-			)
-		)
-		(connect_pads yes
-			(clearance 0)
-		)
-		(min_thickness 0.0254)
-		(filled_areas_thickness no)
-		(fill yes
-			(thermal_gap 0.5)
-			(thermal_bridge_width 0.5)
-			(island_removal_mode 1)
-			(island_area_min 10)
-		)
-		(polygon
-			(pts
-				(xy 141.300879 83.189724) (xy 141.406878 83.020125) (xy 141.246613 82.963041) (xy 140.834153 83.029471)
-				(xy 140.82877 83.155)
-			)
-		)
-	)
-	(zone
 		(net 1)
 		(net_name "GND")
@@
 		(name "$teardrop_padvia$")
 		(hatch none 0.1)
-		(priority 30061)
+		(priority 30059)
 		(attr
 			(teardrop
@@
 		(name "$teardrop_padvia$")
 		(hatch none 0.1)
-		(priority 30060)
+		(priority 30058)
 		(attr
 			(teardrop
@@
 	)
 	(zone
-		(net 4)
-		(net_name "SWC")
-		(layer "F.Cu")
-		(name "$teardrop_padvia$")
-		(hatch none 0.1)
-		(priority 30053)
-		(attr
-			(teardrop
-				(type padvia)
-			)
-		)
-		(connect_pads yes
-			(clearance 0)
-		)
-		(min_thickness 0.0254)
-		(filled_areas_thickness no)
-		(fill yes
-			(thermal_gap 0.5)
-			(thermal_bridge_width 0.5)
-			(island_removal_mode 1)
-			(island_area_min 10)
-		)
-		(polygon
-			(pts
-				(xy 141.377093 82.60442) (xy 141.367625 82.404645) (xy 140.832031 82.405) (xy 140.834002 82.530047)
-				(xy 141.229356 82.63645)
-			)
-		)
-	)
-	(zone
 		(net 5)
 		(net_name "D-")
@@
 		(name "$teardrop_padvia$")
 		(hatch none 0.1)
-		(priority 30054)
+		(priority 30053)
 		(attr
 			(teardrop
@@
 		(name "$teardrop_padvia$")
 		(hatch none 0.1)
-		(priority 30062)
+		(priority 30060)
 		(attr
 			(teardrop
@@
 		(name "$teardrop_padvia$")
 		(hatch none 0.1)
-		(priority 30058)
+		(priority 30056)
 		(attr
 			(teardrop
@@
 		(name "$teardrop_padvia$")
 		(hatch none 0.1)
-		(priority 30059)
+		(priority 30057)
 		(attr
 			(teardrop
@@
 		(hatch edge 0.5)
 		(connect_pads
-			(clearance 0.25)
+			(clearance 0.21)
 		)
-		(min_thickness 0.25)
+		(min_thickness 0.21)
 		(filled_areas_thickness no)
 		(fill yes
-			(thermal_gap 0.25)
-			(thermal_bridge_width 0.25)
+			(thermal_gap 0.21)
+			(thermal_bridge_width 0.21)
 		)
 		(polygon

Commit message: Updated readme + design
Parts:
- removed J3: DEVPGM, Connector_PinHeader_2.54mm:PinHeader_1x04_P2.54mm_Vertical
- J1: footprint Connector_USB:USB_C_Receptacle_HRO_TYPE-C-31-M-12 -> cnhardware:USB_C_MOD_Receptacle_HRO_TYPE-C-31-M-12
- moved R6 0.16 mm to (150.0, 80.0)
- moved C1 0.15 mm to (148.6, 79.6)
- moved Q1 0.05 mm to (133.5, 85.2)
- moved R7 0.05 mm to (136.6, 81.1)
Routing:
- net GND: track 211.5 -> 215.4 mm
