File: hardware/ch570funprog.kicad_pcb (KiCad board)
At the start: 2 copper layers, 34.5 x 12.4 mm, 21 parts, among them J1 USB_C_Receptacle_USB2.0, J2 PGM, Q1 PMOS-SI2301CDS-T1-GE3, U1 USBLC6-2SC6, U2 AMS1117-3.3, U3 CH570Q, Y1 32M

Commit message: Update design
Routing:
- net GND: track 215.4 -> 213.1 mm
Other:
- board text added: "0"
- board text added: "3"
- board text added: "5"
- board text added: "C"
- board text added: "D"
- board text added: "SWCLK"
- board text added: "SWDIO"
- board text removed: "3V3"
- board text removed: "SWC"
- board text removed: "SWD"
