File: hardware/ch570funprog.kicad_pcb (KiCad board)
At the start: 2 copper layers, 34.5 x 12.4 mm, 21 parts, among them J1 USB_C_Receptacle_USB2.0, J2 PGM, Q1 PMOS-SI2301CDS-T1-GE3, U1 USBLC6-2SC6, U2 AMS1117-3.3, U3 CH570Q, Y1 32M

Commit message: Update to rev A
Parts:
- J2: footprint Connector_PinHeader_2.54mm:PinHeader_1x05_P2.54mm_Horizontal -> cnhardware:EDGE_02x04_2.54mm; moved to B.Cu
- moved J2 5.18 mm to (152.1, 82.2), turned to 90 degrees
- moved R6 1.95 mm to (148.1, 79.5), turned to 90 degrees
- moved D1 1.78 mm to (138.1, 85.8)
- moved C1 1.24 mm to (149.8, 79.5)
- moved R5 0.60 mm to (147.1, 79.5), turned to -90 degrees
- moved U2 0.15 mm to (146.5, 84.0)
Connections:
- J2 pad 1: GND -> PSWITCHED
- J2 pad 2: SWD -> VDD
- J2 pad 4: VDD -> SWC
- J2 pad 5: PSWITCHED -> SWD
Routing:
- net GND: track 213.1 -> 203.5 mm, vias 35 -> 46
- net SWC: track 15.0 -> 16.4 mm, vias 2 -> 4
- net +5V: track 21.6 -> 23.0 mm
- net VDD: track 22.3 -> 21.2 mm, vias 2 -> 0
- net PSWITCHED: track 19.1 -> 18.4 mm, vias 0 -> 1
- net SWD: track 15.0 -> 15.2 mm, vias 2 -> 3
Other:
- board size 34.5 x 12.4 mm -> 35.2 x 10.9 mm
- board text added: "1.6mm Thick Non-Lead HASL"
- board text added: "5.0V"
- board text added: "RX"
- board text added: "SCL"
- board text added: "SDA"
- board text added: "SWC"
- board text added: "SWD"
- board text added: "TX"
- board text removed: "0"
- board text removed: "1.0 or 0.8mm thick"
- board text removed: "3"
- board text removed: "5"
- board text removed: "5V"
- board text removed: "C"
- board text removed: "D"
- board text removed: "SWCLK"
- board text removed: "SWDIO"

Commit message: Bump design
Parts:
- moved C1 1.24 mm to (148.6, 79.8), turned to 180 degrees
- moved C3 0.92 mm to (139.7, 85.8)
- moved C4 0.92 mm to (140.7, 85.8)
- moved C5 0.92 mm to (140.2, 84.4)
- moved C6 0.92 mm to (137.2, 79.8)
- moved J2 0.92 mm to (151.2, 82.3)
- moved R5 0.92 mm to (146.2, 79.5)
- moved R6 0.92 mm to (147.2, 79.5), turned to -90 degrees
- moved R7 0.92 mm to (135.7, 81.1)
- moved U2 0.92 mm to (145.6, 84.0)
- moved U3 0.92 mm to (138.4, 82.0)
- moved Y1 0.92 mm to (142.6, 79.1)
- moved R3 0.82 mm to (136.4, 84.7), turned to -90 degrees
- moved C2 0.64 mm to (134.8, 81.1), turned to -90 degrees
- moved D1 0.46 mm to (137.6, 85.8)
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Routing:
- net GND: track 203.5 -> 209.3 mm, vias 46 -> 42
- net PCTL: track 6.92 -> 5.72 mm
- net D-: track 13.4 -> 12.5 mm
- net D+: track 11.9 -> 10.9 mm
- net PSWITCHED: track 18.4 -> 17.7 mm
- net VDD: track 21.2 -> 20.6 mm
Other:
- board size 35.2 x 10.9 mm -> 34.3 x 10.9 mm
