File: hardware/ch570funprog.kicad_pcb (KiCad board)
At the start: 2 copper layers, 34.3 x 10.9 mm, 23 parts, among them J1 USB_C_Receptacle_USB2.0, J2 PGM, Q1 PMOS-SI2301CDS-T1-GE3, U1 USBPROT, U2 AMS1117-3.3, U3 CH570Q, Y1 32M

Commit message: Fix connectivity
Connections:
- C6 pad 2: VDDUC -> +5V
- R7 pad 2: VDDUC -> +5V
- U3 pad 1: VDDUC -> +5V
Routing:
- net +5V: track 23.4 -> 29.2 mm, vias 3 -> 4
- net GND: track 198.3 -> 195.1 mm, vias 42 -> 43
- net VDDUC: track 2.57 -> 0.00 mm
Other:
- board text added: "ch570funprog rev B"
- board text removed: "ch570funprog rev A"

Commit message: Fixup keepout
Parts:
- added JP1: BOOT, Jumper:SolderJumper-2_P1.3mm_Open_RoundedPad1.0x1.5mm, B.Cu at (135.6, 82.4)
- added R8: 5.1k, Resistor_SMD:R_0402_1005Metric, F.Cu at (135.1, 83.3)
- moved R4 1.33 mm to (136.2, 84.8)
- moved R3 0.70 mm to (137.1, 84.8)
- moved D1 0.70 mm to (138.3, 85.7)
- moved Q1 0.18 mm to (133.5, 85.3)
- moved R2 0.14 mm to (130.2, 84.1)
- moved U1 0.14 mm to (131.5, 81.9)
- moved R7 0.13 mm to (135.8, 81.1)
- moved C2 0.12 mm to (134.9, 81.1)
- moved C6 0.08 mm to (137.3, 79.8)
Connections:
- C2 pad 2: Net-(U3-V5) -> +5V
- C6 pad 2: +5V -> PROC33
- R7 pad 1: Net-(U3-V5) -> +5V
- R7 pad 2: +5V -> PROC33
- U3 pad 1: +5V -> PROC33
- U3 pad 2: Net-(U3-V5) -> +5V
Routing:
- net PROC33: track 0.00 -> 2.57 mm
- net GND: track 195.1 -> 192.9 mm, vias 43 -> 42
- net Net-(U3-V5): track 2.16 -> 0.00 mm
- net PCTL: track 5.72 -> 6.57 mm
- net Net-(JP1-A): track 0.00 -> 0.62 mm, vias 0 -> 2
- net +5V: track 29.2 -> 28.7 mm, vias 4 -> 3
- net PSWITCHED: track 17.7 -> 18.1 mm, vias 1 -> 3

Commit message: Bump design
Parts:
- moved J2 0.10 mm to (151.3, 82.3)
Routing:
- net GND: track 192.9 -> 202.5 mm
- net Net-(JP1-A): vias 2 -> 1
Other:
- board size 34.3 x 10.9 mm -> 34.6 x 10.9 mm
