File: hardware/ch570funprog.kicad_sch (KiCad schematic)
At the start: 22 parts, among them J1 USB_C_Receptacle_USB2.0, J2 PGM, J3 DEVPGM, Q1 PMOS-SI2301CDS-T1-GE3, U1 USBLC6-2SC6, U2 AMS1117-3.3, U3 CH570Q, Y1 32M

Commit message: Updated readme + design
Parts:
- J1: footprint Connector_USB:USB_C_Receptacle_HRO_TYPE-C-31-M-12 -> cnhardware:USB_C_MOD_Receptacle_HRO_TYPE-C-31-M-12
Changed lines of the file:
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@@
 			)
 		)
-		(property "Footprint" "Connector_USB:USB_C_Receptacle_HRO_TYPE-C-31-M-12"
+		(property "Footprint" "cnhardware:USB_C_MOD_Receptacle_HRO_TYPE-C-31-M-12"
 			(at 73.66 102.87 0)
 			(effects
