File: hardware/ch570funprog.kicad_sch (KiCad schematic)
At the start: 22 parts, among them J1 USB_C_Receptacle_USB2.0, J2 PGM, J3 DEVPGM, Q1 PMOS-SI2301CDS-T1-GE3, U1 USBLC6-2SC6, U2 AMS1117-3.3, U3 CH570Q, Y1 32M

Commit message: Update to rev A
Parts:
- removed J2: PGM, Connector_PinHeader_2.54mm:PinHeader_1x05_P2.54mm_Horizontal, symbol Connector_Generic:Conn_01x05
- removed J3: DEVPGM, Connector_PinHeader_2.54mm:PinHeader_1x04_P2.54mm_Vertical, symbol Connector_Generic:Conn_01x04
- added J2: PGM, cnhardware:EDGE_02x04_2.54mm, symbol Connector_Generic:Conn_02x04_Odd_Even
- U1: value USBLC6-2SC6 -> USBPROT; LCSC C2687116 -> C558418
Connections:
- net GND: now also J2.7 (Pin_7), J2.8 (Pin_8)
- net PSWITCHED: now also J2.1 (Pin_1)
- net SWC: now also J2.3 (Pin_3), J2.4 (Pin_4)
- net SWD: now also J2.5 (Pin_5), J2.6 (Pin_6)
- net VDD: now also J2.2 (Pin_2)
Other:
- note added: "USB Protection Options: SRV05-4 - C558418 USBLC6-2SC6 - C2687116"
- moved on the sheet: R5, R6

Commit message: Prep for reupload with tooling holes
Parts:
- added H1, H2: Tooling Hole, cnhardware:ToolingHole_JLCPCB, symbol Mechanical:MountingHole

Commit message: Fix connectivity
Connections:
- net VDDUC is gone; now on net +5V: C6.2, R7.2, U3.1 (VDD33/VIO33)
Changed lines of the file:
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@@
+	)
+	(junction
+		(at 68.58 55.88)
+		(diameter 0)
+		(color 0 0 0 0)
 	)
 	(junction
@@
 	(wire
 		(pts
-			(xy 66.04 55.88) (xy 72.39 55.88)
+			(xy 66.04 55.88) (xy 68.58 55.88)
 		)
 		(stroke
@@
 	(wire
 		(pts
+			(xy 68.58 55.88) (xy 72.39 55.88)
+		)
+		(stroke
+			(width 0)
+			(type default)
+		)
+	)
+	(wire
+		(pts
 			(xy 167.64 55.88) (xy 167.64 58.42)
 		)
@@
 		(property "Intersheetrefs" "${INTERSHEET_REFS}"
 			(at 225.252 106.68 0)
-			(hide yes)
-			(show_name no)
-			(do_not_autoplace no)
-			(effects
-				(font
-					(size 1.27 1.27)
-				)
-				(justify right)
-			)
-		)
-	)
-	(global_label "VDDUC"
-		(shape input)
-		(at 66.04 55.88 180)
-		(fields_autoplaced yes)
-		(effects
-			(font
-				(size 1.27 1.27)
-			)
-			(justify right)
-		)
-		(property "Intersheetrefs" "${INTERSHEET_REFS}"
-			(at 56.8257 55.88 0)
 			(hide yes)
 			(show_name no)
@@
 					(unit 1)
 				)
+			)
+		)
+	)
+	(symbol
+		(lib_id "power:+5V")
+		(at 68.58 55.88 0)
+		(unit 1)
+		(body_style 1)
+		(exclude_from_sim no)
+		(in_bom yes)
+		(on_board yes)
+		(in_pos_files yes)
+		(dnp no)
+		(property "Reference" "#PWR026"
+			(at 68.58 59.69 0)
+			(hide yes)
+			(show_name no)
+			(do_not_autoplace no)
+			(effects
+				(font
+					(size 1.27 1.27)
+				)
+			)
+		)
+		(property "Value" "+5V"
+			(at 68.58 48.768 90)
+			(show_name no)
+			(do_not_autoplace no)
+			(effects
+				(font
+					(size 1.27 1.27)
+				)
+				(justify right)
+			)
+		)
+		(property "Footprint" ""
+			(at 68.58 55.88 0)
+			(hide yes)
+			(show_name no)
+			(do_not_autoplace no)
+			(effects
+				(font
+					(size 1.27 1.27)
+				)
+			)
+		)
+		(property "Datasheet" ""
+			(at 68.58 55.88 0)
+			(hide yes)
+			(show_name no)
+			(do_not_autoplace no)
+			(effects
+				(font
+					(size 1.27 1.27)
+				)
+			)
+		)
+		(property "Description" ""
+			(at 68.58 55.88 0)
+			(hide yes)
+			(show_name no)
+			(do_not_autoplace no)
+			(effects
+				(font
+					(size 1.27 1.27)
+				)
+			)
+		)
+		(pin "1"
+		)
+		(instances
+			(project "ch570funprog"
+				(path "/8b3ca9c1-ec01-472e-975f-b13c767b5c47"
+					(reference "#PWR026")
+					(unit 1)
+				)

Commit message: Fixup keepout
Parts:
- added JP1: BOOT, Jumper:SolderJumper-2_P1.3mm_Open_RoundedPad1.0x1.5mm, symbol Jumper:Jumper_2_Open
- added R8: 5.1k, Resistor_SMD:R_0402_1005Metric, symbol Device:R
Connections:
- net +5V: now also C2.2, R7.1, U3.2 (V5), JP1.2 (B); no longer C6.2, R7.2, U3.1 (VDD33/VIO33)
- net D+: now also R8.2
- new net: JP1.1 (A), R8.1
- new net PROC33: C6.2, R7.2, U3.1 (VDD33/VIO33)
