File: hardware-withuart/ch570funprog-withuart.kicad_pcb (KiCad board)
At the start: 2 copper layers, 34.6 x 10.9 mm, 27 parts, among them J1 USB_C_Receptacle_USB2.0, J2 PGM, Q1 PMOS-SI2301CDS-T1-GE3, U1 USBPROT, U2 AMS1117-3.3, U4 CH572D, Y1 32M

Commit message: Update undo italics on 570 board
Other:
- board text added: "1.6mm Thick Non-Lead HASL or OSP"
- board text removed: "1.6mm Thick Non-Lead HASL"
